Commit message: day2: add depth camera and GNSS sensors

File: session_6/tb3_sensor_lab/urdf/waffle.urdf (robot description, URDF)
Before this commit: robot waffle, 11 links, 10 joints
Links:
- added link gps_link
Joints:
- added joint gps_joint: type fixed, parent base_link, child gps_link, origin xyz=-0.05 0 0.19 rpy=0 0 0
